File: pcb/MicroZed-IntanInterface-2Layer/JX1_connections.kicad_sch (KiCad schematic)
At the start: 26 parts, among them Q1 BSS138, Q2 BSS138, SW1 SW_MEC_5E, SW2 SW_MEC_5E

Commit message: Updated PCB after v0.22 bug fixes
Parts:
- D10: value LED 4 -> LED3; footprint LED_SMD:LED_0805_2012Metric -> LED_SMD:LED_0603_1608Metric; LCSC C2296 -> C2833058
- D9: value LED 3 -> LED2; footprint LED_SMD:LED_0805_2012Metric -> LED_SMD:LED_0603_1608Metric; LCSC C2296 -> C2833058
- renumbered C9 to C10, C9 to C18, C9 to C7, C9 to C8, R9 to R1, R9 to R2, TP1 to TP11, TP1 to TP12
Connections:
- net LED4 is gone; now on net LED3: JX1.25 (IO_L5N_T0), Q2.1 (G)
- net LED3: no longer JX1.23 (IO_L5P_T0), Q1.1 (G)
- new net LED2: JX1.23 (IO_L5P_T0), Q1.1 (G)

Commit message: Updates for version 1.0 to ship to UMich
Parts:
- C10, C18, C7, C8: value 22uF -> 22uF 25V; LCSC C5672 -> C12891
- C13, C9: footprint Capacitor_SMD:C_0603_1608Metric -> Capacitor_SMD:C_0402_1005Metric; LCSC C66501 -> C307331
- D10, D9: LCSC C2833058 -> C2286
- JP2, PMODH3, PMODV3: now not fitted
- R1: value 1K -> 1k 1%; footprint Resistor_SMD:R_0603_1608Metric -> Resistor_SMD:R_0402_1005Metric; LCSC C21190 -> C11702
- R19, R20: value 100R -> 150 1%; footprint Resistor_SMD:R_0603_1608Metric -> Resistor_SMD:R_0402_1005Metric; LCSC C22775 -> C25082
- R2: value 100R -> 100 1%; footprint Resistor_SMD:R_0603_1608Metric -> Resistor_SMD:R_0402_1005Metric; LCSC C22775 -> C25076
- R21, R24: value 150R -> 150 1%; footprint Resistor_SMD:R_0603_1608Metric -> Resistor_SMD:R_0402_1005Metric; LCSC C22808 -> C25082
- R22, R27: value 3K3 -> 3k; footprint Resistor_SMD:R_0603_1608Metric -> Resistor_SMD:R_0402_1005Metric
- TP11, TP12: footprint Viktor:TestPoint__Drill1.0mm -> TestPoint:TestPoint_THTPad_D2.0mm_Drill1.0mm
