File: pcb/KiCad-Project/JX1_connections.kicad_sch (KiCad schematic)
At the start: 26 parts, among them Q1 BSS138, Q2 BSS138, SW1 SW_MEC_5E, SW2 SW_MEC_5E

Commit message: PCB revision 1.1 - fixes issues with power supplies.
Parts:
- removed PMODH3: ~, Viktor:PMOD_Socket_Horizontal, symbol Viktor_symbols:PMOD_socket
- removed SW1, SW2: SW_MEC_5E, Viktor:Switch-TH_4P-L6.0-W6.0-P4.50-LS6.5, symbol Switch:SW_MEC_5E
- added ADC1, ADC2, DAC1, DAC2: Conn_Coaxial_Small, Connector_Coaxial:SMA_Amphenol_901-143_Horizontal, symbol Connector:Conn_Coaxial_Small
- added C21, C22, C25: 100nF, Capacitor_SMD:C_0402_1005Metric, symbol Device:C
- added PMODV1: ~, Connector_PinSocket_2.54mm:PinSocket_2x06_P2.54mm_Vertical, symbol Viktor_symbols:PMOD_socket
- added SW1, SW2: SW_Push, Button_Switch_SMD:SW_SPST_TS-1088-xR020, symbol Switch:SW_Push
- added TP1: DAC_VREFIO, TestPoint:TestPoint_THTPad_D2.0mm_Drill1.0mm, symbol Connector:TestPoint
- added U5: DAC70502, Package_SON:Texas_DRX_WSON-10_2.5x2.5mm_P0.5mm, symbol Analog_DAC:DAC70502
- added U6, U9: ADS7029, Package_SO:VSSOP-8_2.3x2mm_P0.5mm, symbol Analog_ADC:ADS7029
- R22, R27: value 3k -> 3.3k; LCSC C22978 -> C25890
Connections:
- net IO_L1N is gone; now on net SWITCH2: JX1.13 (IO_L1N_T0)
- net IO_L1P is gone; now on net SWITCH1: JX1.11 (IO_L1P_T0)
- net IO_L2N is gone; now on net LED3: JX1.14 (IO_L2N_T0)
- net IO_L2P is gone; now on net LED2: JX1.12 (IO_L2P_T0)
- net GND: now also C21.2, C22.2, C25.2, DAC1.2 (Ext), DAC2.2 (Ext), PMODV1.9 (GND), U5.3 (RSTSEL), U5.4 (AGND), U5.5 (SPI2C), U6.8 (GND), U9.8 (GND)
- net IO_L12N: now also PMODV3.7 (IO7)
- net IO_L12P: now also PMODV3.8 (IO8)
- net IO_L14N: now also PMODV3.5 (IO5)
- net IO_L14P: now also PMODV3.6 (IO6)
- net IO_L16N: now also PMODV3.3 (IO3)
- net IO_L16P: now also PMODV3.4 (IO4)
- net IO_L17N: now also PMODV1.6 (IO6)
- net IO_L17P: now also PMODV1.5 (IO5)
- net IO_L18N: now also PMODV3.1 (IO1); no longer PMODV3.7 (IO7)
- net IO_L18P: now also PMODV3.2 (IO2); no longer PMODV3.8 (IO8)
- net IO_L19N: now also PMODV1.2 (IO2)
- net IO_L19P: now also PMODV1.1 (IO1)
- net IO_L21N: now also PMODV1.4 (IO4)
- net IO_L21P: now also PMODV1.3 (IO3)
- net IO_L22N: no longer PMODV3.3 (IO3)
- net IO_L23N: now also PMODV1.8 (IO8)
- net IO_L23P: now also PMODV1.7 (IO7)
- net IO_L24N: no longer PMODV3.1 (IO1)
- net IO_L24P: no longer PMODV3.2 (IO2)
- net LED2: no longer JX1.23 (IO_L5P_T0)
- net LED3: no longer JX1.25 (IO_L5N_T0)
- net SWITCH1: no longer JX1.29 (IO_L7P_T1)
- net SWITCH2: no longer JX1.31 (IO_L7N_T1)
- net VCCIO_34: now also C21.1, C22.1, C25.1, PMODV1.10 (VCC), SW1.1, SW2.1, U5.1 (VDD), U6.1 (DVDD), U6.7 (AVDD), U9.1 (DVDD), U9.7 (AVDD)
- net at R20.2: now also SW2.2
- net at R19.2: now also SW1.2
- net IO_L11P renamed ADC2_NCS
- net ADC2_NCS: now also U9.4 (~{CS})
- net IO_L20N renamed DAC_NSYNC
- net DAC_NSYNC: now also U5.7 (~{SYNC}/A0); no longer PMODV3.5 (IO5)
- net IO_L20P renamed DAC_SDIN
- net DAC_SDIN: now also U5.8 (SDIN/SDA); no longer PMODV3.6 (IO6)
- net IO_L22P renamed DAC_SCLK
- net DAC_SCLK: now also U5.6 (SCLK/SCL); no longer PMODV3.4 (IO4)
- net IO_L8N: no longer names the net of JX1.32 (IO_L8N_T1)
- net IO_L8P: no longer names the net of JX1.30 (IO_L8P_T1)
- net IO_L9N renamed ADC2_SDO
- net ADC2_SDO: now also U9.3 (SDO)
- net IO_L9P renamed ADC2_SCLK
- net ADC2_SCLK: now also U9.2 (SCLK)
- new net: ADC1.2 (Ext), U6.5 (AINM)
- new net: ADC1.1 (In), U6.6 (AINP)
- new net: TP1.1, U5.10 (VREFIO)
- new net: ADC2.2 (Ext), U9.5 (AINM)
- new net: ADC2.1 (In), U9.6 (AINP)
- new net: DAC1.1 (In), U5.2 (VOUTA)
- new net: DAC2.1 (In), U5.9 (VOUTB)
- new net ADC1_NCS: JX1.29 (IO_L7P_T1), U6.4 (~{CS})
- new net ADC1_SCLK: JX1.23 (IO_L5P_T0), U6.2 (SCLK)
- new net ADC1_SDO: JX1.25 (IO_L5N_T0), U6.3 (SDO)
Other:
- note added: "PMODs:"
- note removed: "PMOD3: Single-ended traces 50Ω"
- moved on the sheet: C13, C9, D10, D9, PMODV3, Q1, Q2, R19, R20, R21, R22, R24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
