File: pcb/KiCad-Project/MicroZed-IntanInterface-2Layer.kicad_pcb (KiCad board)
At the start: 4 copper layers, 100.3 x 101.6 mm, 104 parts, among them J1 Screw_Terminal_01x02, J2 Conn_02x05_Odd_Even, J4 USB_C_Receptacle_USB2.0_16P, J7 GND header for probes, Q1 BSS138, Q2 BSS138, Q3 BSS138, Q4 BSS138, SW1 SW_MEC_5E, SW2 SW_MEC_5E, SW3 SW_SPDT, SW4 SW_SPDT, U1 AP331A, U2 TLV62568PDRLR, U3 FT230XS, U9 TLV62568PDRLR

Commit message: PCB revision 1.1 - fixes issues with power supplies.
Parts:
- removed J7: GND header for probes, Connector_PinHeader_2.54mm:PinHeader_1x04_P2.54mm_Vertical
- removed PMODH3: ~, Viktor:PMOD_Socket_Horizontal
- removed REF** (x2): RICE_OWL_LOGO, ELEC327-Kicad:RICE_OWL_LOGO
- added ADC1: Conn_Coaxial_Small, Connector_Coaxial:SMA_Amphenol_901-143_Horizontal, F.Cu at (131.4, 90.2)
- added ADC2: Conn_Coaxial_Small, Connector_Coaxial:SMA_Amphenol_901-143_Horizontal, F.Cu at (131.4, 100.3)
- added C21: 100nF, Capacitor_SMD:C_0402_1005Metric, F.Cu at (123.2, 86.6)
- added C22: 100nF, Capacitor_SMD:C_0402_1005Metric, F.Cu at (123.2, 93.5)
- added C25: 100nF, Capacitor_SMD:C_0402_1005Metric, F.Cu at (113.2, 133.3)
- added DAC1: Conn_Coaxial_Small, Connector_Coaxial:SMA_Amphenol_901-143_Horizontal, F.Cu at (131.4, 125.7)
- added DAC2: Conn_Coaxial_Small, Connector_Coaxial:SMA_Amphenol_901-143_Horizontal, F.Cu at (131.4, 135.9)
- added PMODV1: ~, Connector_PinSocket_2.54mm:PinSocket_2x06_P2.54mm_Vertical, F.Cu at (132.1, 106.7)
- added S1: ~, ELEC327-Kicad:RICE_OWL_LOGO, F.Cu at (46.2, 78.2)
- added S2: ~, ELEC327-Kicad:RICE_OWL_LOGO, B.Cu at (90.7, 112.8)
- added TP1: DAC_VREFIO, TestPoint:TestPoint_THTPad_D2.0mm_Drill1.0mm, B.Cu at (110.0, 133.3)
- added U4: TLV62569DDC, Package_TO_SOT_SMD:SOT-23-6, F.Cu at (80.7, 60.2)
- added U5: DAC70502, Package_SON:Texas_DRX_WSON-10_2.5x2.5mm_P0.5mm, F.Cu at (109.9, 129.0)
- added U6: ADS7029, Package_SO:VSSOP-8_2.3x2mm_P0.5mm, F.Cu at (123.2, 88.9)
- J2: value Conn_02x05_Odd_Even -> Conn_02x04_Odd_Even; footprint Connector_PinSocket_2.54mm:PinSocket_2x05_P2.54mm_Vertical -> Connector_PinSocket_2.54mm:PinSocket_2x04_P2.54mm_Vertical
- R12, R22, R27: value 3k -> 3.3k
- SW1, SW2: value SW_MEC_5E -> SW_Push; footprint Viktor:Switch-TH_4P-L6.0-W6.0-P4.50-LS6.5 -> Button_Switch_SMD:SW_SPST_TS-1088-xR020
- U2: value TLV62568PDRLR -> TLV62569DDC; footprint Package_TO_SOT_SMD:SOT-563 -> Package_TO_SOT_SMD:SOT-23-6
- U9: value TLV62568PDRLR -> ADS7029; footprint Package_TO_SOT_SMD:SOT-563 -> Package_SO:VSSOP-8_2.3x2mm_P0.5mm
- moved J2 77.2 mm to (58.4, 147.3), turned to -90 degrees
- moved U9 44.0 mm to (123.2, 95.8), turned to 0 degrees
- moved SW2 25.7 mm to (130.8, 77.5), turned to 180 degrees
- moved TP11 20.0 mm to (105.2, 87.9), turned to -90 degrees
- moved SW1 16.0 mm to (130.8, 69.3), turned to 180 degrees
- moved U2 15.9 mm to (97.0, 60.2)
- moved R20 15.5 mm to (124.3, 80.0), turned to 90 degrees
- moved C9 15.4 mm to (121.7, 74.2), turned to 90 degrees
- moved R22 14.1 mm to (123.1, 74.2), turned to 90 degrees
- moved R27 14.0 mm to (121.8, 80.0), turned to 90 degrees
- moved Q2 13.6 mm to (119.2, 62.4), turned to 0 degrees
- moved R19 13.0 mm to (124.5, 74.2), turned to 90 degrees
- moved C13 12.8 mm to (123.1, 80.0), turned to 90 degrees
- moved D10 12.6 mm to (133.3, 58.7), turned to -90 degrees
- moved R1 12.3 mm to (115.6, 72.5)
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- renumbered J4 to J8
Connections:
- J2 pad 1: +5V -> GND
- J2 pad 2: +5V -> GND
- J2 pad 4: GND -> +5V
- J2 pad 6: GND -> VCCIO_35
- J2 pad 7: VCCIO_35 -> GND
- J2 pad 8: VCCIO_35 -> VCCIO_34
- JX1 pad 11: /JX1_connections/IO_L1P -> /JX1_connections/SWITCH1
- JX1 pad 12: /JX1_connections/IO_L2P -> /JX1_connections/LED2
- JX1 pad 13: /JX1_connections/IO_L1N -> /JX1_connections/SWITCH2
- JX1 pad 14: /JX1_connections/IO_L2N -> /JX1_connections/LED3
- JX1 pad 23: /JX1_connections/LED2 -> /JX1_connections/ADC1_SCLK
- JX1 pad 25: /JX1_connections/LED3 -> /JX1_connections/ADC1_SDO
- JX1 pad 29: /JX1_connections/SWITCH1 -> /JX1_connections/ADC1_NCS
- JX1 pad 30: /JX1_connections/IO_L8P -> unconnected-(JX1-IO_L8P_T1-Pad30)
- JX1 pad 31: /JX1_connections/SWITCH2 -> unconnected-(JX1-IO_L7N_T1-Pad31)
- JX1 pad 32: /JX1_connections/IO_L8N -> unconnected-(JX1-IO_L8N_T1-Pad32)
- JX1 pad 35: /JX1_connections/IO_L9P -> /JX1_connections/ADC2_SCLK
- JX1 pad 37: /JX1_connections/IO_L9N -> /JX1_connections/ADC2_SDO
- JX1 pad 41: /JX1_connections/IO_L11P -> /JX1_connections/ADC2_NCS
- JX1 pad 68: /JX1_connections/IO_L20P -> /JX1_connections/DAC_SDIN
- JX1 pad 70: /JX1_connections/IO_L20N -> /JX1_connections/DAC_NSYNC
- JX1 pad 74: /JX1_connections/IO_L22P -> /JX1_connections/DAC_SCLK
- PMODV3 pad 1: /JX1_connections/IO_L24N -> /JX1_connections/IO_L18N
- PMODV3 pad 2: /JX1_connections/IO_L24P -> /JX1_connections/IO_L18P
- PMODV3 pad 3: /JX1_connections/IO_L22N -> /JX1_connections/IO_L16N
- PMODV3 pad 4: /JX1_connections/IO_L22P -> /JX1_connections/IO_L16P
- PMODV3 pad 5: /JX1_connections/IO_L20N -> /JX1_connections/IO_L14N
- PMODV3 pad 6: /JX1_connections/IO_L20P -> /JX1_connections/IO_L14P
- PMODV3 pad 7: /JX1_connections/IO_L18N -> /JX1_connections/IO_L12N
- PMODV3 pad 8: /JX1_connections/IO_L18P -> /JX1_connections/IO_L12P
- R11 pad 1: Net-(U9-FB) -> Net-(U2-FB)
- R19 pad 2: Net-(SW1-A) -> Net-(R19-Pad2)
- R20 pad 2: Net-(SW2-A) -> Net-(R20-Pad2)
- R6 pad 2: Net-(U2-FB) -> Net-(U4-FB)
- R8 pad 1: Net-(U2-FB) -> Net-(U4-FB)
- R9 pad 2: Net-(U9-FB) -> Net-(U2-FB)
- SW1 pad 2: VCCIO_34 -> Net-(R19-Pad2)
- SW2 pad 2: VCCIO_34 -> Net-(R20-Pad2)
- U2 pad 3: SW_2V5 -> SW_3V3
- U9 pad 1: /VADJ_EN -> VCCIO_34
- U9 pad 2: GND -> /JX1_connections/ADC2_SCLK
- U9 pad 3: SW_3V3 -> /JX1_connections/ADC2_SDO
- U9 pad 4: +5V -> /JX1_connections/ADC2_NCS
- U9 pad 5: PG_CARRIER -> Net-(ADC2-Ext)
- U9 pad 6: Net-(U9-FB) -> Net-(ADC2-In)
Routing:
- net /JX1_connections/IO_L14N: track 0.00 -> 94.0 mm
- net /JX1_connections/IO_L14P: track 0.00 -> 93.3 mm
- net /JX1_connections/IO_L12N: track 0.00 -> 93.3 mm
- net /JX1_connections/IO_L12P: track 0.00 -> 92.6 mm
- net /JX1_connections/IO_L16N: track 0.00 -> 90.3 mm, vias 0 -> 1
- net /JX1_connections/IO_L16P: track 0.00 -> 89.0 mm, vias 0 -> 1
- net /JX1_connections/IO_L20N: track 88.2 -> 0.00 mm
- net /JX1_connections/IO_L20P: track 87.5 -> 0.00 mm
- net /JX1_connections/IO_L22N: track 83.5 -> 0.00 mm, vias 1 -> 0
- net /JX1_connections/IO_L24N: track 83.4 -> 0.00 mm, vias 1 -> 0
- net /JX1_connections/IO_L22P: track 82.7 -> 0.00 mm, vias 1 -> 0
- net /JX1_connections/IO_L24P: track 82.6 -> 0.00 mm, vias 1 -> 0
- net VCCIO_34: track 251.0 -> 314.4 mm, vias 7 -> 12
- net /JX1_connections/DAC_SDIN: track 0.00 -> 39.3 mm
- net /JX1_connections/DAC_NSYNC: track 0.00 -> 37.5 mm
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Other:
- outline, holes or cut-outs redrawn
- board text added: "Intan Interface Kemere Lab (C) 2026 Rev 1.1"
- board text removed: "Intan Interface Kemere Lab (C) 2026 Rev 1.0"
