File: pcb/KiCad-Project/MicroZed-IntanInterface-2Layer.kicad_sch (KiCad schematic)
At the start: 51 parts, among them J1 Screw_Terminal_01x02, J2 Conn_02x05_Odd_Even, J4 USB_C_Receptacle_USB2.0_16P, J7 GND header for probes, SW3 SW_SPDT, SW4 SW_SPDT, U1 AP331A, U2 TLV62568PDRLR, U9 TLV62568PDRLR

Commit message: PCB revision 1.1 - fixes issues with power supplies.
Parts:
- removed J2: Conn_02x05_Odd_Even, Connector_PinSocket_2.54mm:PinSocket_2x05_P2.54mm_Vertical, symbol Connector_Generic:Conn_02x05_Odd_Even
- removed J7: GND header for probes, Connector_PinHeader_2.54mm:PinHeader_1x04_P2.54mm_Vertical, symbol Connector:Conn_01x04_Pin
- removed U2, U9: TLV62568PDRLR, Package_TO_SOT_SMD:SOT-563, symbol Regulator_Switching:TLV62568DDC
- added J2: Conn_02x04_Odd_Even, Connector_PinSocket_2.54mm:PinSocket_2x04_P2.54mm_Vertical, symbol Connector_Generic:Conn_02x04_Odd_Even
- added S1, S2: ~, ELEC327-Kicad:RICE_OWL_LOGO, symbol ELEC327-Kicad:RICE_OWL
- added U2, U4: TLV62569DDC, Package_TO_SOT_SMD:SOT-23-6, symbol Regulator_Switching:TLV62569DDC
- R12: value 3k -> 3.3k; LCSC C22978 -> C25890
- renumbered J4 to J8
Connections:
- net +5V: now also J2.4 (Pin_4), U2.4 (VIN), U4.4 (VIN)
- net GND: now also J2.1 (Pin_1), J2.2 (Pin_2), J2.3 (Pin_3), J2.5 (Pin_5), J2.7 (Pin_7), U2.2 (GND), U4.2 (GND)
- net PG_CARRIER: now also U2.5 (PG), U4.5 (PG)
- net SW_2V5: now also U4.3 (SW)
- net SW_3V3: now also U2.3 (SW)
- net VADJ_EN: now also U2.1 (EN), U4.1 (EN)
- net VCCIO_34: now also J2.8 (Pin_8)
- net VCCIO_35: now also J2.6 (Pin_6)
- net at R6.2, R8.1: now also U4.6 (FB)
- net at R11.1, R9.2: now also U2.6 (FB)
