File: pcb/glance-carrier/JX1_connections.kicad_sch (KiCad schematic)
At the start: 37 parts, among them Q1 BSS138, Q2 BSS138, SW1 SW_Push, SW2 SW_Push, U5 DAC70502, U6 ADS7029, U9 ADS7029

Commit message: pcb(glance-carrier): rebrand title blocks to the GLANCE name
Sets the title-block title on all schematic sheets and the board to
"GLANCE Project Intan Interface Carrier for MicroZed module" (were the old
"Intan Interface" and Viktor "MicroZed development carrier board" placeholders).
Sheet names and design content unchanged.
Other:
- title: MicroZed development carrier board -> GLANCE Project Intan Interface Carrier for MicroZed module
Changed lines of the file:
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@@
   (paper "A4")
   (title_block
-    (title "MicroZed development carrier board")
+    (title "GLANCE Project Intan Interface Carrier for MicroZed module")
     (date "2023-08-19")
     (rev "4")
