File: pcb/glance-carrier/glance-carrier.kicad_sch (KiCad schematic)
At the start: 52 parts, among them J1 Screw_Terminal_01x02, J2 Conn_02x04_Odd_Even, J8 USB_C_Receptacle_USB2.0_16P, SW3 SW_SPDT, SW4 SW_SPDT, U1 AP331A, U2 TLV62569DDC, U4 TLV62569DDC

Commit message: pcb(glance-carrier): rebrand title blocks to the GLANCE name
Sets the title-block title on all schematic sheets and the board to
"GLANCE Project Intan Interface Carrier for MicroZed module" (were the old
"Intan Interface" and Viktor "MicroZed development carrier board" placeholders).
Sheet names and design content unchanged.
Other:
- title: Intan Interface carrier board -> GLANCE Project Intan Interface Carrier for MicroZed module
Changed lines of the file:
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@@
   (paper "A4")
   (title_block
-    (title "Intan Interface carrier board")
+    (title "GLANCE Project Intan Interface Carrier for MicroZed module")
     (date "2025-08-18")
     (rev "1.0")
